File: USB-OV2640-module.kicad_sch (KiCad schematic)
At the start: 116 parts, among them J1 USB_C_Receptacle_USB2.0_14P, J2 Conn_01x04_Pin, SW1 TS-1088-AR02016, SW2 TS-1088-AR02016, U1 USBLC6-2SC6, U2 XC6206-1.2V, U3 ESP32-S3, U4 XC6206-2.8V, U5 W25Q64JVSSIQ, Y1 XTM25040000JT00351005

Commit message: Rev0 ready
Parts:
- C26: footprint Capacitor_SMD:C_0201_0603Metric -> Capacitor_SMD:C_0402_1005Metric
- R10, R11, R12, R13, R14, R15, R18, R19, R2, R20, R21, R22, R23, R24, R25, R26, R27, R28, R29, R3, R30, R31, R32, R33, R34, R35, R36, R37, R38, R4, R42, R43, R44, R5, R6, R9: footprint PCM_Resistor_SMD_AKL:R_01005_0402Metric -> PCM_Resistor_SMD_AKL:R_0402_1005Metric
- R16, R17, R39, R40, R41: footprint PCM_Resistor_SMD_AKL:R_0201_0603Metric -> PCM_Resistor_SMD_AKL:R_0402_1005Metric
Connections:
- net TWI_SCK is gone; now on net SIO_D: R40.1
- net TWI_SDA is gone; now on net SIO_C: R41.1
- net USB_con+: now also R4.2; no longer R5.2
- net USB_con-: now also R5.2; no longer R4.2
- net USB_filter+: now also FL1.1, U1.1 (I/O1); no longer FL1.4, U1.3 (I/O2)
- net USB_filter-: now also FL1.4, U1.3 (I/O2); no longer FL1.1, U1.1 (I/O1)
- net USB_mcu+: now also FL1.2; no longer FL1.3
- net USB_mcu-: now also FL1.3; no longer FL1.2
- net USB_res+: now also R4.1, U1.6 (I/O1); no longer R5.1, U1.4 (I/O2)
- net USB_res-: now also R5.1, U1.4 (I/O2); no longer R4.1, U1.6 (I/O1)
- net Y2: now also R25.1; no longer R18.1
- net Y3: now also R24.1; no longer R19.1
- net Y4: now also R23.1; no longer R20.1
- net Y5: now also R22.1; no longer R21.1
- net Y6: now also R21.1; no longer R22.1
- net Y7: now also R20.1; no longer R23.1
- net Y8: now also R19.1; no longer R24.1
- net Y9: now also R18.1; no longer R25.1
Other:
- moved on the sheet: FL1
